File: hardware/carrier-board/carrier-board.kicad_sch (KiCad schematic)
At the start: 6 parts, among them U1 STM32G474RET6

Commit message: inicial schematic
Parts:
- removed J_B2B: Main Bus, symbol Connector_Generic:Conn_02x10_Odd_Even
- removed J_SWD: SWD Conn, symbol Connector_Generic:Conn_01x05
- removed J_USB: USB-C, symbol Connector:USB_C_Receptacle_USB2.0_16pin
- removed U1: STM32G474RET6, symbol MCU_ST_STM32G4:STM32G474RETx
- removed U_ESD: USBLC6-2SC6, symbol Protection:USBLC6-2SC6
- removed U_LDO: AP2112K-3.3, symbol Regulator_Linear:AP2112K-3.3TRG1
Other:
- added sheet expansion (expansion.kicad_sch)
- added sheet mcu_core (mcu_core.kicad_sch)
- added sheet peripherals (peripherals.kicad_sch)
- title: STM32G474 Carrier Board - Base -> (none)
Changed lines of the file:
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@@
-(kicad_sch (version 20240108) (generator "gemini-cli-init-script")
-  (paper "A4")
-  (title_block
-    (title "STM32G474 Carrier Board - Base")
-    (date "2026-07-27")
-    (rev "1.0")
-  )
-  (symbol (lib_id "MCU_ST_STM32G4:STM32G474RETx") (at 152.4 101.6 0) (unit 1)
-    (in_bom yes) (on_board yes)
-    (property "Reference" "U1" (at 152.4 96.52 0)
-      (effects (font (size 1.27 1.27)))
-    )
-    (property "Value" "STM32G474RET6" (at 152.4 106.67999999999999 0)
-      (effects (font (size 1.27 1.27)))
-    )
-    (property "Footprint" "" (at 152.4 101.6 0) (effects (font (size 1.27 1.27)) (hide yes)))
-    (property "Datasheet" "" (at 152.4 101.6 0) (effects (font (size 1.27 1.27)) (hide yes)))
-    (property "LCSC" "C913074" (at 152.4 101.6 0)
-      (effects (font (size 1.27 1.27)) (hide yes))
-    )
-  )  (symbol (lib_id "Connector:USB_C_Receptacle_USB2.0_16pin") (at 76.2 76.2 0) (unit 1)
-    (in_bom yes) (on_board yes)
-    (property "Reference" "J_USB" (at 76.2 71.12 0)
-      (effects (font (size 1.27 1.27)))
-    )
-    (property "Value" "USB-C" (at 76.2 81.28 0)
-      (effects (font (size 1.27 1.27)))
-    )
-    (property "Footprint" "" (at 76.2 76.2 0) (effects (font (size 1.27 1.27)) (hide yes)))
-    (property "Datasheet" "" (at 76.2 76.2 0) (effects (font (size 1.27 1.27)) (hide yes)))
-    (property "LCSC" "C167339" (at 76.2 76.2 0)
-      (effects (font (size 1.27 1.27)) (hide yes))
-    )
-  )  (symbol (lib_id "Regulator_Linear:AP2112K-3.3TRG1") (at 76.2 127 0) (unit 1)
-    (in_bom yes) (on_board yes)
-    (property "Reference" "U_LDO" (at 76.2 121.92 0)
-      (effects (font (size 1.27 1.27)))
-    )
-    (property "Value" "AP2112K-3.3" (at 76.2 132.08 0)
-      (effects (font (size 1.27 1.27)))
-    )
-    (property "Footprint" "" (at 76.2 127 0) (effects (font (size 1.27 1.27)) (hide yes)))
-    (property "Datasheet" "" (at 76.2 127 0) (effects (font (size 1.27 1.27)) (hide yes)))
-    (property "LCSC" "C84949" (at 76.2 127 0)
-      (effects (font (size 1.27 1.27)) (hide yes))
-    )
-  )  (symbol (lib_id "Connector_Generic:Conn_01x05") (at 228.6 76.2 0) (unit 1)
-    (in_bom yes) (on_board yes)
-    (property "Reference" "J_SWD" (at 228.6 71.12 0)
-      (effects (font (size 1.27 1.27)))
-    )
-    (property "Value" "SWD Conn" (at 228.6 81.28 0)
-      (effects (font (size 1.27 1.27)))
-    )
-    (property "Footprint" "" (at 228.6 76.2 0) (effects (font (size 1.27 1.27)) (hide yes)))
-    (property "Datasheet" "" (at 228.6 76.2 0) (effects (font (size 1.27 1.27)) (hide yes)))
-    (property "LCSC" "C2897385" (at 228.6 76.2 0)
-      (effects (font (size 1.27 1.27)) (hide yes))
-    )
-  )  (symbol (lib_id "Connector_Generic:Conn_02x10_Odd_Even") (at 228.6 127 0) (unit 1)
-    (in_bom yes) (on_board yes)
-    (property "Reference" "J_B2B" (at 228.6 121.92 0)
-      (effects (font (size 1.27 1.27)))
-    )
-    (property "Value" "Main Bus" (at 228.6 132.08 0)
-      (effects (font (size 1.27 1.27)))
-    )
-    (property "Footprint" "" (at 228.6 127 0) (effects (font (size 1.27 1.27)) (hide yes)))
-    (property "Datasheet" "" (at 228.6 127 0) (effects (font (size 1.27 1.27)) (hide yes)))
-    (property "LCSC" "C2922180" (at 228.6 127 0)
-      (effects (font (size 1.27 1.27)) (hide yes))
-    )
-  )  (symbol (lib_id "Protection:USBLC6-2SC6") (at 101.6 76.2 0) (unit 1)
-    (in_bom yes) (on_board yes)
-    (property "Reference" "U_ESD" (at 101.6 71.12 0)
-      (effects (font (size 1.27 1.27)))
-    )
-    (property "Value" "USBLC6-2SC6" (at 101.6 81.28 0)
-      (effects (font (size 1.27 1.27)))
-    )
-    (property "Footprint" "" (at 101.6 76.2 0) (effects (font (size 1.27 1.27)) (hide yes)))
-    (property "Datasheet" "" (at 101.6 76.2 0) (effects (font (size 1.27 1.27)) (hide yes)))
-    (property "LCSC" "C87327" (at 101.6 76.2 0)
-      (effects (font (size 1.27 1.27)) (hide yes))
-    )
-  )
+(kicad_sch
+	(version 20260306)
+	(generator "eeschema")
+	(generator_version "10.0")
+	(paper "A4")
+	(sheet
+		(at 152.4 241.3)
+		(size 203.2 127)
+		(exclude_from_sim no)
+		(in_bom yes)
+		(on_board yes)
+		(dnp no)
+		(stroke
+			(width 0)
+			(type solid)
+		)
+		(fill
+			(color 0 0 0 0)
+		)
+		(property "Sheetname" "mcu_core"
+			(at 152.4 238 0)
+			(show_name no)
+			(do_not_autoplace no)
+			(effects
+				(font
+					(size 3.556 3.556)
+				)
+			)
+		)
+		(property "Sheetfile" "mcu_core.kicad_sch"
+			(at 0 0 0)
+			(hide yes)
+			(show_name no)
+			(do_not_autoplace no)
+			(effects
+				(font
+					(size 1.27 1.27)
+				)
+			)
+		)
+		(instances
+			(project "carrier-board"
+				(path "/a1b2c3d4-e5f6-4a1b-9c8d-7e6f5a4b3c2d"
+					(page "3")
+				)
+			)
+		)
+	)
+	(sheet
+		(at 406.4 101.6)
+		(size 203.2 127)
+		(exclude_from_sim no)
+		(in_bom yes)
+		(on_board yes)
+		(dnp no)
+		(stroke
+			(width 0)
+			(type solid)
+		)
+		(fill
+			(color 0 0 0 0)
+		)
+		(property "Sheetname" "peripherals"
+			(at 406.4 98 0)
+			(show_name no)
+			(do_not_autoplace no)
+			(effects
+				(font
+					(size 3.556 3.556)
+				)
+			)
+		)
+		(property "Sheetfile" "peripherals.kicad_sch"
+			(at 0 0 0)
+			(hide yes)
+			(show_name no)
+			(do_not_autoplace no)
+			(effects
+				(font
+					(size 1.27 1.27)
+				)
+			)
+		)
+		(instances
+			(project "carrier-board"
+				(path "/a1b2c3d4-e5f6-4a1b-9c8d-7e6f5a4b3c2d"
+					(page "4")
+				)
+			)
+		)
+	)
+	(sheet
+		(at 406.4 241.3)
+		(size 203.2 127)
+		(exclude_from_sim no)
+		(in_bom yes)
+		(on_board yes)
+		(dnp no)
+		(stroke
+			(width 0)
+			(type solid)
+		)
+		(fill
+			(color 0 0 0 0)
+		)
+		(property "Sheetname" "expansion"
+			(at 406.4 238 0)
+			(show_name no)
+			(do_not_autoplace no)
+			(effects
+				(font
+					(size 3.556 3.556)
+				)
+			)
+		)
+		(property "Sheetfile" "expansion.kicad_sch"
+			(at 0 0 0)
+			(hide yes)
+			(show_name no)
+			(do_not_autoplace no)
+			(effects
+				(font
+					(size 1.27 1.27)
+				)
+			)
+		)
+		(instances
+			(project "carrier-board"
+				(path "/a1b2c3d4-e5f6-4a1b-9c8d-7e6f5a4b3c2d"
+					(page "5")
+				)
+			)
+		)
+	)
+	(sheet_instances
+		(path "/"
+			(page "1")
+		)
+	)
+	(embedded_fonts no)
 )
