File: hardware/carrier-board/mcu_core.kicad_sch (KiCad schematic)
At the start: 20 parts, among them J1 DIN41612_02x08_AB_EvenPins, J2 DIN41612_02x08_AB_EvenPins, J3 TC2030, J4 Conn_01x04_Socket, J5 Conn_01x04_Pin, J6 USB_C_Receptacle_USB2.0_16P, SW1 SW_Push, U1 STM32G474RETx, U2 AMS1117-3.3, Y1 Crystal_GND3

Commit message: sch review
Parts:
- removed J1: DIN41612_02x08_AB_EvenPins, Connector_PinSocket_2.00mm:PinSocket_2x08_P2.00mm_Vertical_SMD, symbol Connector:DIN41612_02x08_AB_EvenPins
- added C10, C4, C5: 10uF, Capacitor_SMD:C_0805_2012Metric, symbol Device:C
- added C11, C12, C6, C7, C8, C9: 100nF, Capacitor_SMD:C_0805_2012Metric, symbol Device:C
- added C3: 100nf, Capacitor_SMD:C_0603_1608Metric, symbol Device:C
- added R10, R11: 22K, Resistor_SMD:R_0805_2012Metric, symbol Device:R
- added R12: 10k, Resistor_SMD:R_0805_2012Metric, symbol Device:R
- added R8, R9: 5.1k, Resistor_SMD:R_0805_2012Metric, symbol Device:R
- added TP1, TP2, TP3, TP4: TestPoint, TestPoint:TestPoint_Pad_D1.0mm, symbol Connector:TestPoint
- C1, C2: value C -> 22pf; footprint Capacitor_SMD:C_0603_1608Metric -> C_0805_2012Metric
Connections:
- net +3.3V: now also J2.b8 (Pin_b8), C10.1, C4.1, C6.1, C7.1, C8.1, C9.1, R10.1, R11.1, TP1.1, TP3.1; no longer J2.b6 (Pin_b6)
- net +5V: now also J2.b4 (Pin_b4), C5.1, TP2.1; no longer J2.b10 (Pin_b10)
- net GND: now also J2.b2 (Pin_b2), C10.2, C11.1, C12.1, C3.2, C4.2, C5.2, C6.2, C7.2, C8.2, C9.2, R12.1, R8.2, R9.2
- net HWID_0: now also U1.8 (PC0)
- net HWID_1: now also U1.9 (PC1)
- net HWID_2: now also U1.10 (PC2)
- net HWID_3: now also U1.11 (PC3)
- net HWID_A: now also U1.12 (PA0)
- net RESET: now also R1.2, SW1.2, C3.1
- net SCL: now also U1.43 (PA9), R10.2
- net SDA: now also U1.42 (PA8), R11.2
- net USB_D+: now also J6.B6 (D+); no longer J6.B7 (D-)
- net USB_D-: now also J6.B7 (D-); no longer J6.A6 (D+)
- net SPI_CS / PWM: now reaches J2.a2 (Pin_a2)
- net SPI_CS / PWM: now also U1.18 (PA4)
- net SPI_MOSI / PWM: now reaches J2.a4 (Pin_a4)
- net SPI_MOSI / PWM: now also U1.21 (PA7)
- net SPI_MISO / PWM: now reaches J2.a6 (Pin_a6)
- net SPI_MISO / PWM: now also U1.20 (PA6)
- net SPI_SCK / PWM: now reaches J2.a8 (Pin_a8)
- net SPI_SCK / PWM: now also U1.19 (PA5)
- net TRT_GPIO_3: now reaches J2.b16 (Pin_b16)
- net TRT_GPIO_3: now also U1.17 (PA3)
- net at FB1.2, U1.29 (VDDA): now also C11.2, C12.2, TP4.1
- net TRT_GPIO_1: now reaches U1.13 (PA1)
- net TRT_GPIO_1: now also J2.b6 (Pin_b6)
- net TRT_GPIO_2: now reaches U1.14 (PA2)
- net TRT_GPIO_2: now also J2.b10 (Pin_b10)
- net at U1.60 (PB7): now also R12.2
- net at J6.A5 (CC1): now also R8.1
- net at J6.B5 (CC2): now also R9.1
Other:
- note added: "necesito reemplazar esto por un controld egpio para las resistencias"
- moved on the sheet: C1, C2, J2, R1, SW1, Y1

Commit message: feat(hardware): finalize schematic, update README and set initial PCB layout
Parts:
- added C13: 100nf, Capacitor_SMD:C_0603_1608Metric, symbol Device:C
- added D1, D2: LED, LED_SMD:LED_0805_2012Metric, symbol Device:LED
- added D3: 1N5819HW, Diode_SMD:D_SOD-123, symbol Diode:1N5819
- added J1: Conn_01x02_Pin, Connector_PinHeader_2.54mm:PinHeader_1x02_P2.54mm_Vertical, symbol Connector:Conn_01x02_Pin
- added Q1: AO3400A, Package_TO_SOT_SMD:SOT-23, symbol Transistor_FET:AO3400A
- added R13: 1k, Resistor_SMD:R_0805_2012Metric, symbol Device:R
- added R14: 470, Resistor_SMD:R_0805_2012Metric, symbol Device:R
- added R15: 10k, Resistor_SMD:R_0805_2012Metric, symbol Device:R
- added R16: 100, Resistor_SMD:R_0805_2012Metric, symbol Device:R
- FB1: footprint (none) -> L_0805_2012Metric
- R10, R11: value 22K -> 2.2K
Connections:
- net +3.3V: now also J2.8 (Pin_8), U1.1 (VBAT), U1.32 (VDD), U1.48 (VDD), U1.64 (VDD), R13.1; no longer J2.b8 (Pin_b8), R10.1, R11.1
- net +5V: now also J2.4 (Pin_4), C13.1, D3.1 (K), D3.2 (A), J1.1 (Pin_1), J1.2 (Pin_2), Q1.3 (D); no longer J2.b4 (Pin_b4)
- net GND: now also J2.2 (Pin_2), C13.2, D1.1 (K), D2.1 (K), Q1.2 (S), R15.2; no longer J2.b2 (Pin_b2)
- net HWID_0: now also J2.9 (Pin_9); no longer J2.a10 (Pin_a10)
- net HWID_1: now also J2.11 (Pin_11); no longer J2.a12 (Pin_a12)
- net HWID_2: now also J2.13 (Pin_13); no longer J2.a14 (Pin_a14)
- net HWID_3: now also J2.15 (Pin_15); no longer J2.a16 (Pin_a16)
- net SCL: now also J2.14 (Pin_14), U1.61 (PB8); no longer J2.b14 (Pin_b14), U1.43 (PA9)
- net SDA: now also J2.12 (Pin_12), U1.62 (PB9); no longer J2.b12 (Pin_b12), U1.42 (PA8)
- net SPI_CS / PWM: now also J2.1 (Pin_1), U1.59 (PB6); no longer J2.a2 (Pin_a2), U1.18 (PA4)
- net SPI_MISO / PWM: now also J2.5 (Pin_5); no longer J2.a6 (Pin_a6)
- net SPI_MOSI / PWM: now also J2.3 (Pin_3); no longer J2.a4 (Pin_a4)
- net SPI_SCK / PWM: now also J2.7 (Pin_7), R14.1; no longer J2.a8 (Pin_a8)
- net TRT_GPIO_1: now also J2.6 (Pin_6); no longer J2.b6 (Pin_b6)
- net TRT_GPIO_2: now also J2.10 (Pin_10), U1.18 (PA4); no longer J2.b10 (Pin_b10), U1.14 (PA2)
- net TRT_GPIO_3: now also J2.16 (Pin_16), U1.24 (PB0); no longer J2.b16 (Pin_b16), U1.17 (PA3)
- net I2C_PU_EN: now reaches U1.4 (PC15)
- net I2C_PU_EN: now also R10.1, R11.1
- net Vm_out: now reaches U1.57 (PB4)
- net Vm_out: now also R16.1
- new net: Q1.1 (G), R15.1, R16.2
- new net: D2.2 (A), R14.2
- new net: D1.2 (A), R13.2
Other:
- note removed: "necesito reemplazar esto por un controld egpio para las resistencias"
- moved on the sheet: C4, C5, R10, R11, R12, TP1, TP2, U2

Commit message: pcb placement
Parts:
- J5: footprint Connector_PinHeader_2.00mm:PinHeader_1x04_P2.00mm_Horizontal -> 303C-321018-30-04:303C-321018-30-04
- SW1: footprint Button_Switch_THT:SW_PUSH_1P1T_6x3.5mm_H5.0_APEM_MJTP1250 -> Button_Switch_SMD:SW_SPST_B3U-1000P-B
Connections:
- net at C1.1, U1.5 (PF0): now also Y1.2; no longer Y1.1
- net at C2.1, U1.6 (PF1): now also Y1.1; no longer Y1.2
Changed lines of the file:
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@@
 	)
 	(junction
-		(at 74.93 82.55)
-		(diameter 0)
-		(color 0 0 0 0)
-	)
-	(junction
 		(at 107.95 36.83)
 		(diameter 0)
@@
 	)
 	(junction
+		(at 74.93 82.55)
+		(diameter 0)
+		(color 0 0 0 0)
+	)
+	(junction
 		(at 237.49 149.86)
 		(diameter 0)
@@
 	)
 	(symbol
+		(lib_id "Device:Crystal_GND3")
+		(at 78.74 82.55 0)
+		(mirror y)
+		(unit 1)
+		(body_style 1)
+		(exclude_from_sim no)
+		(in_bom yes)
+		(on_board yes)
+		(in_pos_files yes)
+		(dnp no)
+		(property "Reference" "Y1"
+			(at 78.74 82.296 90)
+			(show_name no)
+			(do_not_autoplace no)
+			(effects
+				(font
+					(size 1.27 1.27)
+				)
+			)
+		)
+		(property "Value" "Crystal_GND3"
+			(at 79.248 89.154 0)
+			(show_name no)
+			(do_not_autoplace no)
+			(effects
+				(font
+					(size 1.27 1.27)
+				)
+			)
+		)
+		(property "Footprint" "Crystal:Crystal_SMD_5032-4Pin_5.0x3.2mm"
+			(at 78.74 82.55 0)
+			(hide yes)
+			(show_name no)
+			(do_not_autoplace no)
+			(effects
+				(font
+					(size 1.27 1.27)
+				)
+			)
+		)
+		(property "Datasheet" ""
+			(at 78.74 82.55 0)
+			(hide yes)
+			(show_name no)
+			(do_not_autoplace no)
+			(effects
+				(font
+					(size 1.27 1.27)
+				)
+			)
+		)
+		(property "Description" "Three pin crystal, GND on pin 3"
+			(at 78.74 82.55 0)
+			(hide yes)
+			(show_name no)
+			(do_not_autoplace no)
+			(effects
+				(font
+					(size 1.27 1.27)
+				)
+			)
+		)
+		(pin "1"
+		)
+		(pin "2"
+		)
+		(pin "3"
+		)
+		(instances
+			(project "carrier-board"
+				(path "/a1b2c3d4-e5f6-4a1b-9c8d-7e6f5a4b3c2d/c3d4e5f6-a1b2-4c3d-9e8f-5a4b3c2d1e7a"
+					(reference "Y1")
+					(unit 1)
+				)
+			)
+		)
+	)
+	(symbol
 		(lib_id "Connector:DIN41612_02x08_AB_EvenPins")
 		(at 252.73 31.75 0)
@@
 			)
 		)
-		(property "Footprint" "Connector_PinHeader_2.00mm:PinHeader_1x04_P2.00mm_Horizontal"
+		(property "Footprint" "303C-321018-30-04:303C-321018-30-04"
 			(at 264.16 64.77 0)
 			(hide yes)
@@
 			)
 		)
-		(property "Footprint" "Button_Switch_THT:SW_PUSH_1P1T_6x3.5mm_H5.0_APEM_MJTP1250"
+		(property "Footprint" "Button_Switch_SMD:SW_SPST_B3U-1000P-B"
 			(at 33.02 114.3 0)
 			(hide yes)
@@
 					(unit 1)
 				)
-			)
-		)
-	)
-	(symbol
-		(lib_id "Device:Crystal_GND3")
-		(at 78.74 82.55 0)
-		(unit 1)
-		(body_style 1)
-		(exclude_from_sim no)
-		(in_bom yes)
-		(on_board yes)
-		(in_pos_files yes)
-		(dnp no)
-		(property "Reference" "Y1"
-			(at 78.74 82.296 90)
-			(show_name no)
-			(do_not_autoplace no)
-			(effects
-				(font
-					(size 1.27 1.27)
-				)
-			)
-		)
-		(property "Value" "Crystal_GND3"
-			(at 78.232 89.154 0)
-			(show_name no)
-			(do_not_autoplace no)
-			(effects
-				(font
-					(size 1.27 1.27)
-				)
-			)
-		)
-		(property "Footprint" "Crystal:Crystal_SMD_5032-4Pin_5.0x3.2mm"
-			(at 78.74 82.55 0)
-			(hide yes)
-			(show_name no)
-			(do_not_autoplace no)
-			(effects
-				(font
-					(size 1.27 1.27)
-				)
-			)
-		)
-		(property "Datasheet" ""
-			(at 78.74 82.55 0)
-			(hide yes)
-			(show_name no)
-			(do_not_autoplace no)
-			(effects
-				(font
-					(size 1.27 1.27)
-				)
-			)
-		)
-		(property "Description" "Three pin crystal, GND on pin 3"
-			(at 78.74 82.55 0)
-			(hide yes)
-			(show_name no)
-			(do_not_autoplace no)
-			(effects
-				(font
-					(size 1.27 1.27)
-				)
-			)
-		)
-		(pin "1"
-		)
-		(pin "2"
-		)
-		(pin "3"
-		)
-		(instances
-			(project "carrier-board"
-				(path "/a1b2c3d4-e5f6-4a1b-9c8d-7e6f5a4b3c2d/c3d4e5f6-a1b2-4c3d-9e8f-5a4b3c2d1e7a"
-					(reference "Y1")
-					(unit 1)
-				)
